Commit message: add Husky-Panda controller

File: husky_panda_description/urdf/husky_panda copy.urdf (robot description, URDF)
Before this commit: robot panda, 23 links, 22 joints
Links:
- removed link world
- added link base_footprint
- added link base_link; collision box size=0.7899200000000001 0.5709 0.10375; collision box size=0.9874 0.5709 0.12375
- added link front_left_wheel_link, mass 2.637; collision cylinder length=0.1143 radius=0.1651; visual mesh filename=package://husky_description/meshes/wheel.dae
- added link front_right_wheel_link, mass 2.637; collision cylinder length=0.1143 radius=0.1651; visual mesh filename=package://husky_description/meshes/wheel.dae
- added link imu_link
- added link inertial_link, mass 46.034
- added link rear_bumper_link; visual mesh filename=package://husky_description/meshes/bumper.dae
- added link rear_left_wheel_link, mass 2.637; collision cylinder length=0.1143 radius=0.1651; visual mesh filename=package://husky_description/meshes/wheel.dae
- added link rear_right_wheel_link, mass 2.637; collision cylinder length=0.1143 radius=0.1651; visual mesh filename=package://husky_description/meshes/wheel.dae
- added link top_chassis_link; visual mesh filename=package://husky_description/meshes/top_chassis.dae
- added link top_structure_link; collision box size=0.38992 0.56 1.3; visual mesh filename=package://husky_description/meshes/roas_dyros.STL
- added link user_rail_link; visual mesh filename=package://husky_description/meshes/user_rail.dae
- link panda_hand: geometry collision mesh filename=package://franka_description/meshes/collision/hand.stl; visual mesh filename=package://franka_description/meshes/visual/hand.dae
- link panda_leftfinger: geometry collision box size=17.5e-3 15.2e-3 18.5e-3; collision box size=17.5e-3 7e-3 23.5e-3
- link panda_link0: geometry collision mesh filename=package://franka_description/meshes/collision/link0.stl; visual mesh filename=package://franka_description/meshes/visual/link0.dae
- link panda_link1: geometry collision mesh filename=package://franka_description/meshes/collision/link1.stl; visual mesh filename=package://franka_description/meshes/visual/link1.dae
- link panda_link2: geometry collision mesh filename=package://franka_description/meshes/collision/link2.stl; visual mesh filename=package://franka_description/meshes/visual/link2.dae
- link panda_link3: geometry collision mesh filename=package://franka_description/meshes/collision/link3.stl; visual mesh filename=package://franka_description/meshes/visual/link3.dae
- link panda_link4: geometry collision mesh filename=package://franka_description/meshes/collision/link4.stl; visual mesh filename=package://franka_description/meshes/visual/link4.dae
- link panda_link5: geometry collision mesh filename=package://franka_description/meshes/collision/link5.stl; visual mesh filename=package://franka_description/meshes/visual/link5.dae
- link panda_link6: geometry collision mesh filename=package://franka_description/meshes/collision/link6.stl; visual mesh filename=package://franka_description/meshes/visual/link6.dae
- link panda_link7: geometry collision mesh filename=package://franka_description/meshes/collision/link7.stl; visual mesh filename=package://franka_description/meshes/visual/link7.dae
- link panda_rightfinger: geometry collision box size=17.5e-3 15.2e-3 18.5e-3; collision box size=17.5e-3 7e-3 23.5e-3
Joints:
- removed joint world_joint
- added joint base_footprint_joint: type fixed, parent base_link, child base_footprint, origin xyz=0 0 -0.13228 rpy=0 0 0
- added joint front_left_wheel: type continuous, parent base_link, child front_left_wheel_link, origin xyz=0.256 0.2854 0.03282 rpy=0 0 0, axis 0 1 0
- added joint front_right_wheel: type continuous, parent base_link, child front_right_wheel_link, origin xyz=0.256 -0.2854 0.03282 rpy=0 0 0, axis 0 1 0
- added joint imu_joint: type fixed, parent base_link, child imu_link, origin xyz=0.19 0 0.149 rpy=0 -1.5708 3.1416
- added joint inertial_joint: type fixed, parent base_link, child inertial_link, origin xyz=0 0 0 rpy=0 0 0
- added joint panda_joint_base_link: type fixed, parent base_link, child panda_link0, origin xyz=0.3 0.0 0.256 rpy=0.0 0.0 0.0
- added joint rear_bumper: type fixed, parent base_link, child rear_bumper_link, origin xyz=-0.48 0 0.091 rpy=0 0 3.14159
- added joint rear_left_wheel: type continuous, parent base_link, child rear_left_wheel_link, origin xyz=-0.256 0.2854 0.03282 rpy=0 0 0, axis 0 1 0
- added joint rear_right_wheel: type continuous, parent base_link, child rear_right_wheel_link, origin xyz=-0.256 -0.2854 0.03282 rpy=0 0 0, axis 0 1 0
- added joint top_chassis_joint: type fixed, parent base_link, child top_chassis_link
- added joint top_structure_joint: type fixed, parent base_link, child top_structure_link, origin xyz=0 0 0 rpy=0 0 0
- added joint user_rail: type fixed, parent base_link, child user_rail_link, origin xyz=0.272 0 0.245 rpy=0 0 0
